File: Kicad/Shield_Nucleo144/Shield_Nucleo144.kicad_pcb (KiCad board)
At the start: 2 copper layers, 133.1 x 146 mm, 64 parts, among them IC1 DW01A, J1 5V, J10 PCB_Déporté, J11 Transistor_Bypass, J12 Transistor_Bypass, J13 Transistor_Bypass, J14 5V, J15 I2C1, J16 Hard_Reset, J17 Batterie, J18 Panneau_Solaire, J19 5V, J2 3.3V, J20 I2C1, J21 Anémomètre, J22 SPI4, J23 5V, J24 I2C2, J26 Transistor_Bypass, J27 Transistor_Bypass, J28 5V, J29 I2C2, J3 I2C1, J30 Foudre, J31 5V, J32 I2C2, J33 Pluviomètre, J37 Transistor_Bypass, J39 5V, J4 UART1, J40 I2C2, J41 5V, J43 5V, J45 5V, J5 UART3, J6 UART7, J7 5V, J8 I2C1, J9 3.3V, Q12 GPS, Q2 ESP, Q3 DHT, Q4 Anémomètre, Q5 FS8205A, Q8 Pluviomètre, Q9 Sky_Temperature, U1 TP4056, U2 MIC2288YD5-TR, U3 ESP8266-12E/ESP-12E

Commit message: Add files via upload
Parts:
- removed J16: Hard_Reset, Connector_JST:JST_EH_B2B-EH-A_1x02_P2.50mm_Vertical
Connections:
- A1 pad CN11_14: Hard_Reset_In -> unconnected-(A1-PadCN11_14)
- U3 pad 1: Hard_Reset_In -> unconnected-(U3-Pad1)
Routing:
- net Hard_Reset_In: track 234.6 -> 0.00 mm, vias 2 -> 0
- net I2C1_SDA: track 173.0 -> 181.5 mm
