File: Kicad/Shield_Nucleo144/Shield_Nucleo144.kicad_sch (KiCad schematic)
At the start: 64 parts, among them IC1 DW01A, J1 5V, J10 PCB_Déporté, J11 Transistor_Bypass, J12 Transistor_Bypass, J13 Transistor_Bypass, J14 5V, J15 I2C1, J16 Hard_Reset, J17 Batterie, J18 Panneau_Solaire, J19 5V, J2 3.3V, J20 I2C1, J21 Anémomètre, J22 SPI4, J23 5V, J24 I2C2, J26 Transistor_Bypass, J27 Transistor_Bypass, J28 5V, J29 I2C2, J3 I2C1, J30 Foudre, J31 5V, J32 I2C2, J33 Pluviomètre, J37 Transistor_Bypass, J39 5V, J4 UART1, J40 I2C2, J41 5V, J43 5V, J45 5V, J5 UART3, J6 UART7, J7 5V, J8 I2C1, J9 3.3V, Q12 GPS, Q2 ESP, Q3 DHT, Q4 Anémomètre, Q5 FS8205A, Q8 Pluviomètre, Q9 Sky_Temperature, U1 TP4056, U2 MIC2288YD5-TR, U3 ESP8266-12E/ESP-12E

Commit message: Add files via upload
Parts:
- removed J16: Hard_Reset, Connector_JST:JST_EH_B2B-EH-A_1x02_P2.50mm_Vertical, symbol Connector:Conn_01x02_Male
Connections:
- net Hard_Reset_In: no longer names the net of A1.CN11_14 (RESET)
- net Hard_Reset_In: no longer U3.1 (RESET)
Changed lines of the file:
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@@
     (stroke (width 0) (type default) (color 0 0 0 0))
   )
-  (wire (pts (xy 104.14 256.54) (xy 104.14 257.81))
-    (stroke (width 0) (type default) (color 0 0 0 0))
-  )
   (wire (pts (xy 199.39 228.6) (xy 199.39 224.79))
     (stroke (width 0) (type default) (color 0 0 0 0))
@@
     (stroke (width 0) (type default) (color 0 0 0 0))
   )
-  (wire (pts (xy 95.25 256.54) (xy 104.14 256.54))
-    (stroke (width 0) (type default) (color 0 0 0 0))
-  )
   (wire (pts (xy 132.08 85.09) (xy 124.46 85.09))
     (stroke (width 0) (type default) (color 0 0 0 0))
@@
     (stroke (width 0) (type default) (color 0 0 0 0))
   )
-  (wire (pts (xy 95.25 254) (xy 101.6 254))
-    (stroke (width 0) (type default) (color 0 0 0 0))
-  )
   (wire (pts (xy 59.69 345.44) (xy 57.15 345.44))
     (stroke (width 0) (type default) (color 0 0 0 0))
@@
     )
   )
-  (global_label "Hard_Reset_In" (shape input) (at 101.6 254 0) (fields_autoplaced)
-    (effects (font (size 1.27 1.27)) (justify left))
-    (property "Intersheet References" "${INTERSHEET_REFS}" (id 0) (at 117.3179 253.9206 0)
-      (effects (font (size 1.27 1.27)) (justify left) hide)
-    )
-  )
-  (global_label "Hard_Reset_In" (shape input) (at 233.68 52.07 180) (fields_autoplaced)
-    (effects (font (size 1.27 1.27)) (justify right))
-    (property "Intersheet References" "${INTERSHEET_REFS}" (id 0) (at 217.9621 52.1494 0)
-      (effects (font (size 1.27 1.27)) (justify right) hide)
-    )
-  )
-  (global_label "Hard_Reset_In" (shape input) (at 513.08 162.56 180) (fields_autoplaced)
-    (effects (font (size 1.27 1.27)) (justify right))
-    (property "Intersheet References" "${INTERSHEET_REFS}" (id 0) (at 497.3621 162.6394 0)
-      (effects (font (size 1.27 1.27)) (justify right) hide)
-    )
-  )
   (global_label "UART1_RX" (shape input) (at 33.02 185.42 0) (fields_autoplaced)
     (effects (font (size 1.27 1.27)) (justify left))
@@
     (pin "1")
   )
-  (symbol (lib_id "power:GND") (at 104.14 257.81 0) (unit 1)
-    (in_bom yes) (on_board yes) (fields_autoplaced)
-    (property "Reference" "#PWR020" (id 0) (at 104.14 264.16 0)
-      (effects (font (size 1.27 1.27)) hide)
-    )
-    (property "Value" "GND" (id 1) (at 104.14 262.89 0))
-    (property "Footprint" "" (id 2) (at 104.14 257.81 0)
-      (effects (font (size 1.27 1.27)) hide)
-    )
-    (property "Datasheet" "" (id 3) (at 104.14 257.81 0)
-      (effects (font (size 1.27 1.27)) hide)
-    )
-    (pin "1")
-  )
   (symbol (lib_id "power:GND") (at 354.33 134.62 0) (unit 1)
     (in_bom yes) (on_board yes) (fields_autoplaced)
@@
     (pin "2")
   )
-  (symbol (lib_id "Connector:Conn_01x02_Male") (at 90.17 254 0) (unit 1)
-    (in_bom yes) (on_board yes) (fields_autoplaced)
-    (property "Reference" "J16" (id 0) (at 90.805 248.92 0))
-    (property "Value" "Hard_Reset" (id 1) (at 90.805 251.46 0))
-    (property "Footprint" "Connector_JST:JST_EH_B2B-EH-A_1x02_P2.50mm_Vertical" (id 2) (at 90.17 254 0)
-      (effects (font (size 1.27 1.27)) hide)
-    )
-    (property "Datasheet" "~" (id 3) (at 90.17 254 0)
-      (effects (font (size 1.27 1.27)) hide)
-    )
-    (pin "1")
-    (pin "2")
-  )
   (symbol (lib_id "power:+5V") (at 175.26 185.42 0) (unit 1)
     (in_bom yes) (on_board yes) (fields_autoplaced)
@@
       (reference "#PWR019") (unit 1) (value "GND") (footprint "")
     )
-    (path "/328fc78b-8879-4bf5-8be3-e3cc4f7d7a5f"
-      (reference "#PWR020") (unit 1) (value "GND") (footprint "")
-    )
     (path "/881805b7-c25f-4aa8-a00c-3aa1d7fdccbe"
       (reference "#PWR021") (unit 1) (value "+5V") (footprint "")
@@
       (reference "J15") (unit 1) (value "I2C1") (footprint "Connector_JST:JST_EH_B2B-EH-A_1x02_P2.50mm_Vertical")
     )
-    (path "/d66dca5b-4327-49b6-8a1d-705aed354741"
-      (reference "J16") (unit 1) (value "Hard_Reset") (footprint "Connector_JST:JST_EH_B2B-EH-A_1x02_P2.50mm_Vertical")
-    )
     (path "/154ecdf3-080d-4190-99bc-aeee22026525"
