File: Kicad/Shield_Raspy/Shield_Raspy.kicad_sch (KiCad schematic)
At the start: 4 parts, among them J1 Raspberry_Pi_2_3, K1 HEADER_FEMALE_5x2_1.27mm_SMD, U1 CO2, U2 NUCLEO-L432KC

Commit message: Add files via upload
Connections:
- net +5V: now also J1.4 (5V), U2.CN4_4 (+5V)
- net GND: now also J1.14 (GND), J1.20 (GND), J1.25 (GND), J1.30 (GND), J1.34 (GND), J1.39 (GND), J1.9 (GND), U2.CN3_4 (GND_CN3)
Changed lines of the file:
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@@
 (kicad_sch (version 20211123) (generator eeschema)
   (paper "A4")
+  (junction (at 241.3 88.9) (diameter 0) (color 0 0 0 0)
+  )
+  (junction (at 251.46 88.9) (diameter 0) (color 0 0 0 0)
+  )
+  (junction (at 248.92 88.9) (diameter 0) (color 0 0 0 0)
+  )
+  (junction (at 254 88.9) (diameter 0) (color 0 0 0 0)
+  )
+  (junction (at 256.54 88.9) (diameter 0) (color 0 0 0 0)
+  )
+  (junction (at 246.38 22.86) (diameter 0) (color 0 0 0 0)
+  )
+  (junction (at 243.84 88.9) (diameter 0) (color 0 0 0 0)
+  )
+  (junction (at 246.38 88.9) (diameter 0) (color 0 0 0 0)
+  )
   (no_connect (at 36.83 97.79))
   (no_connect (at 36.83 95.25))
@@
     (stroke (width 0) (type solid) (color 0 0 0 0))
   )
+  (wire (pts (xy 143.51 34.29) (xy 143.51 31.75))
+    (stroke (width 0) (type default) (color 0 0 0 0))
+  )
   (wire (pts (xy 35.56 90.17) (xy 36.83 90.17))
     (stroke (width 0) (type solid) (color 0 0 0 0))
@@
     (stroke (width 0) (type solid) (color 0 0 0 0))
   )
+  (wire (pts (xy 78.74 64.77) (xy 81.28 64.77))
+    (stroke (width 0) (type default) (color 0 0 0 0))
+  )
   (wire (pts (xy 44.45 90.17) (xy 44.45 87.63))
     (stroke (width 0) (type solid) (color 0 0 0 0))
@@
     (stroke (width 0) (type default) (color 0 0 0 0))
   )
+  (wire (pts (xy 254 88.9) (xy 256.54 88.9))
+    (stroke (width 0) (type default) (color 0 0 0 0))
+  )
   (wire (pts (xy 241.3 88.9) (xy 241.3 93.98))
     (stroke (width 0) (type default) (color 0 0 0 0))
@@
     (stroke (width 0) (type default) (color 0 0 0 0))
   )
+  (wire (pts (xy 81.28 64.77) (xy 81.28 67.31))
+    (stroke (width 0) (type default) (color 0 0 0 0))
+  )
   (wire (pts (xy 227.33 33.02) (xy 231.14 33.02))
     (stroke (width 0) (type default) (color 0 0 0 0))
   )
+  (wire (pts (xy 251.46 88.9) (xy 254 88.9))
+    (stroke (width 0) (type default) (color 0 0 0 0))
+  )
   (wire (pts (xy 45.72 52.07) (xy 48.26 52.07))
     (stroke (width 0) (type default) (color 0 0 0 0))
   )
+  (wire (pts (xy 256.54 88.9) (xy 259.08 88.9))
+    (stroke (width 0) (type default) (color 0 0 0 0))
+  )
   (wire (pts (xy 45.72 46.99) (xy 48.26 46.99))
     (stroke (width 0) (type default) (color 0 0 0 0))
   )
+  (wire (pts (xy 246.38 88.9) (xy 248.92 88.9))
+    (stroke (width 0) (type default) (color 0 0 0 0))
+  )
+  (wire (pts (xy 246.38 22.86) (xy 248.92 22.86))
+    (stroke (width 0) (type default) (color 0 0 0 0))
+  )
   (wire (pts (xy 34.29 100.33) (xy 36.83 100.33))
     (stroke (width 0) (type solid) (color 0 0 0 0))
   )
+  (wire (pts (xy 243.84 88.9) (xy 246.38 88.9))
+    (stroke (width 0) (type default) (color 0 0 0 0))
+  )
   (wire (pts (xy 142.24 64.77) (xy 144.78 64.77))
     (stroke (width 0) (type default) (color 0 0 0 0))
@@
     (stroke (width 0) (type default) (color 0 0 0 0))
   )
+  (wire (pts (xy 241.3 88.9) (xy 243.84 88.9))
+    (stroke (width 0) (type default) (color 0 0 0 0))
+  )
   (wire (pts (xy 46.99 116.84) (xy 46.99 114.3))
     (stroke (width 0) (type default) (color 0 0 0 0))
@@
     (stroke (width 0) (type solid) (color 0 0 0 0))
   )
+  (wire (pts (xy 248.92 88.9) (xy 251.46 88.9))
+    (stroke (width 0) (type default) (color 0 0 0 0))
+  )
   (wire (pts (xy 246.38 22.86) (xy 246.38 19.05))
     (stroke (width 0) (type default) (color 0 0 0 0))
@@
   (wire (pts (xy 41.91 97.79) (xy 44.45 97.79))
     (stroke (width 0) (type solid) (color 0 0 0 0))
+  )
+  (wire (pts (xy 142.24 34.29) (xy 143.51 34.29))
+    (stroke (width 0) (type default) (color 0 0 0 0))
   )
   (wire (pts (xy 109.22 57.15) (xy 111.76 57.15))
@@
   (symbol (lib_id "power:+5V") (at 44.45 87.63 0) (unit 1)
     (in_bom yes) (on_board yes) (fields_autoplaced)
-    (property "Reference" "#PWR?" (id 0) (at 44.45 91.44 0)
+    (property "Reference" "#PWR0101" (id 0) (at 44.45 91.44 0)
       (effects (font (size 1.27 1.27)) hide)
     )
@@
     )
     (pin "1")
+    (pin "10")
     (pin "2")
     (pin "3")
+    (pin "4")
     (pin "5")
+    (pin "6")
     (pin "7")
+    (pin "8")
     (pin "9")
-    (pin "10")
-    (pin "8")
-    (pin "6")
-    (pin "4")
   )
   (symbol (lib_id "power:+5V") (at 35.56 87.63 0) (unit 1)
     (in_bom yes) (on_board yes) (fields_autoplaced)
-    (property "Reference" "#PWR?" (id 0) (at 35.56 91.44 0)
+    (property "Reference" "#PWR0102" (id 0) (at 35.56 91.44 0)
       (effects (font (size 1.27 1.27)) hide)
     )
@@
     )
     (property "Datasheet" "" (id 3) (at 35.56 87.63 0)
+      (effects (font (size 1.27 1.27)) hide)
+    )
+    (pin "1")
+  )
+  (symbol (lib_id "power:GND") (at 81.28 67.31 0) (unit 1)
+    (in_bom yes) (on_board yes) (fields_autoplaced)
+    (property "Reference" "#PWR0103" (id 0) (at 81.28 73.66 0)
+      (effects (font (size 1.27 1.27)) hide)
+    )
+    (property "Value" "GND" (id 1) (at 81.28 72.39 0))
+    (property "Footprint" "" (id 2) (at 81.28 67.31 0)
+      (effects (font (size 1.27 1.27)) hide)
+    )
+    (property "Datasheet" "" (id 3) (at 81.28 67.31 0)
+      (effects (font (size 1.27 1.27)) hide)
+    )
+    (pin "1")
+  )
+  (symbol (lib_id "power:+5V") (at 143.51 31.75 0) (unit 1)
+    (in_bom yes) (on_board yes) (fields_autoplaced)
+    (property "Reference" "#PWR?" (id 0) (at 143.51 35.56 0)
+      (effects (font (size 1.27 1.27)) hide)
+    )
+    (property "Value" "+5V" (id 1) (at 143.51 26.67 0))
+    (property "Footprint" "" (id 2) (at 143.51 31.75 0)
+      (effects (font (size 1.27 1.27)) hide)
+    )
+    (property "Datasheet" "" (id 3) (at 143.51 31.75 0)
       (effects (font (size 1.27 1.27)) hide)
     )
@@
     )
     (path "/9f2393b9-1bc9-4155-8b89-027d363b4770"
+      (reference "#PWR0101") (unit 1) (value "+5V") (footprint "")
+    )
+    (path "/d400635d-f7bf-472d-9e60-3223427ef8f1"
+      (reference "#PWR0102") (unit 1) (value "+5V") (footprint "")
+    )
+    (path "/d4c93017-bd96-47e4-9b43-467e505f10b8"
+      (reference "#PWR0103") (unit 1) (value "GND") (footprint "")
+    )
+    (path "/eb9c01b6-c066-4481-a500-c414ae593ed3"
       (reference "#PWR?") (unit 1) (value "+5V") (footprint "")
     )
-    (path "/d400635d-f7bf-472d-9e60-3223427ef8f1"
-      (reference "#PWR?") (unit 1) (value "+5V") (footprint "")
-    )
